File: vga/hw/vga/vga.kicad_pcb (KiCad board)
At the start: 2 copper layers, 99.1 x 99.1 mm, 25 parts, among them J1 ISP, J2 VGA, J3 PWR, U1 74HC74, U10 74HC590, U11 74HC590, U2 ATmega328-PU, U3 74HC00, U4 74HC04, U5 74HC74, U6 CY7C199, U7 74HC245, U8 74HC161, U9 74HC166, X1 DOTCLK

Commit message: flesh out PCB
Parts:
- added C10: 100n, Capacitor_THT:C_Disc_D3.4mm_W2.1mm_P2.50mm, F.Cu at (149.2, 105.0)
- added C11: 100n, Capacitor_THT:C_Disc_D3.4mm_W2.1mm_P2.50mm, F.Cu at (116.2, 122.8)
- added C12: 100n, Capacitor_THT:C_Disc_D3.4mm_W2.1mm_P2.50mm, F.Cu at (116.2, 82.1)
- added C13: 100n, Capacitor_THT:C_Disc_D3.4mm_W2.1mm_P2.50mm, F.Cu at (131.4, 61.8)
- added C14: 100n, Capacitor_THT:C_Disc_D3.4mm_W2.1mm_P2.50mm, F.Cu at (149.2, 120.2)
- added C15: 100n, Capacitor_THT:C_Disc_D3.4mm_W2.1mm_P2.50mm, F.Cu at (159.4, 140.6)
- added C16: 100n, Capacitor_THT:C_Disc_D3.4mm_W2.1mm_P2.50mm, F.Cu at (116.2, 102.5)
- added C17: 100n, Capacitor_THT:C_Disc_D3.4mm_W2.1mm_P2.50mm, F.Cu at (139.1, 120.2)
- added C19: 100µ, Capacitor_THT:CP_Radial_D6.3mm_P2.50mm, F.Cu at (159.4, 64.4)
- added C5: 100n, Capacitor_THT:C_Disc_D3.4mm_W2.1mm_P2.50mm, F.Cu at (128.9, 120.2)
- added C7: 100n, Capacitor_THT:C_Disc_D3.4mm_W2.1mm_P2.50mm, F.Cu at (139.1, 105.0)
- added C8: 100n, Capacitor_THT:C_Disc_D3.4mm_W2.1mm_P2.50mm, F.Cu at (116.2, 61.8)
- added C9: 100n, Capacitor_THT:C_Disc_D3.4mm_W2.1mm_P2.50mm, F.Cu at (101.0, 61.8)
- added J4: BUS, Connector_PinHeader_2.54mm:PinHeader_2x08_P2.54mm_Vertical, F.Cu at (139.1, 64.4)
- added U12: 74HC590, Package_SO:SOIC-16_3.9x9.9mm_P1.27mm, F.Cu at (126.4, 112.6)
- added U13: 74HC590, Package_SO:SOIC-16_3.9x9.9mm_P1.27mm, F.Cu at (126.4, 127.9)
- added U14: 74HC574, Package_SO:SOIC-20W_7.5x12.8mm_P1.27mm, F.Cu at (111.1, 92.3)
- added U15: 74HC574, Package_SO:SOIC-20W_7.5x12.8mm_P1.27mm, F.Cu at (111.1, 112.6)
- added U16: 74LS138, Package_SO:SOIC-16_3.9x9.9mm_P1.27mm, F.Cu at (146.7, 112.6)
- added U17: 74HC574, Package_SO:SOIC-20W_7.5x12.8mm_P1.27mm, F.Cu at (95.9, 72.0)
- C6: value 100µ -> 100n; footprint Capacitor_THT:CP_Radial_D6.3mm_P2.50mm -> Capacitor_THT:C_Disc_D3.4mm_W2.1mm_P2.50mm
- J2: value VGA -> PWR; footprint Connector_Dsub:DSUB-9_Female_Horizontal_P2.77x2.84mm_EdgePinOffset4.94mm_Housed_MountingHolesOffset7.48mm -> Connector_PinHeader_2.54mm:PinHeader_1x04_P2.54mm_Vertical
- J3: value PWR -> VGA; footprint Connector_PinHeader_2.54mm:PinHeader_1x04_P2.54mm_Vertical -> Connector_Dsub:DSUB-15-HD_Female_Horizontal_P2.29x1.98mm_EdgePinOffset3.03mm_Housed_MountingHolesOffset4.94mm
- R1, R2: footprint Resistor_THT:R_Axial_DIN0309_L9.0mm_D3.2mm_P12.70mm_Horizontal -> Resistor_THT:R_Axial_DIN0204_L3.6mm_D1.6mm_P7.62mm_Horizontal
- U10: value 74HC590 -> 74HC574; footprint Package_SO:SOIC-16_3.9x9.9mm_P1.27mm -> Package_SO:SOIC-20W_7.5x12.8mm_P1.27mm
- U11: value 74HC590 -> 74HC166
- U2: footprint Package_DIP:DIP-28_W7.62mm -> Package_DIP:DIP-28_W7.62mm_Socket
- U6: value CY7C199 -> 74HC74; footprint Package_DIP:DIP-28_W7.62mm_Socket -> Package_SO:SOIC-14_3.9x8.7mm_P1.27mm
- U7: value 74HC245 -> CY7C199; footprint Package_SO:SOIC-20W_7.5x12.8mm_P1.27mm -> Package_DIP:DIP-28_W7.62mm_Socket
- U8: value 74HC161 -> 74HC245; footprint Package_SO:SOIC-16_3.9x9.9mm_P1.27mm -> Package_SO:SOIC-20W_7.5x12.8mm_P1.27mm
- U9: value 74HC166 -> 74HC161
- moved C3 113.9 mm to (149.2, 135.5), turned to 180 degrees
- moved C4 106.8 mm to (139.0, 135.5), turned to 180 degrees
- moved J3 102.6 mm to (108.6, 145.6), turned to 0 degrees
- moved C1 100.0 mm to (128.9, 135.5), turned to 180 degrees
- moved R1 93.9 mm to (151.8, 79.6), turned to 90 degrees
- moved D1 89.9 mm to (151.8, 64.4), turned to 180 degrees
- moved J1 85.5 mm to (159.4, 112.6), turned to 0 degrees
- moved U5 85.2 mm to (136.5, 127.9)
- moved U2 83.1 mm to (156.8, 72.0)
- moved U6 82.8 mm to (146.7, 143.1)
- moved X1 81.8 mm to (156.8, 132.9)
- moved U1 81.2 mm to (136.5, 143.1)
- moved U4 74.6 mm to (146.7, 127.9)
- moved U8 71.8 mm to (111.1, 132.9)
- moved U3 68.1 mm to (146.7, 97.4)
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- renumbered C5 to C18
Connections:
- J2 pad 1: Net-(J2-Pad1) -> +5V
- J2 pad 2: Net-(J2-Pad1) -> GND
- J2 pad 3: Net-(J2-Pad1) -> GND
- J2 pad 4: (no net) -> +5V
- J3 pad 1: +5V -> Net-(J3-Pad1)
- J3 pad 2: GND -> Net-(J3-Pad1)
- J3 pad 3: GND -> Net-(J3-Pad1)
- J3 pad 4: +5V -> (no net)
- R2 pad 1: Net-(J2-Pad1) -> Net-(J3-Pad1)
- U10 pad 1: /C1 -> /~EXTEN
- U10 pad 10: /~RSTCOUNT -> GND
- U10 pad 11: /~CSTART -> /~WRLADDR
- U10 pad 12: /~VIS -> /R1
- U10 pad 13: /DOTCLK -> /R0
- U10 pad 14: /EXTEN -> /C5
- U10 pad 15: /C0 -> /C4
- U10 pad 16: +5V -> /C3
- U10 pad 2: /C2 -> /D0
- U10 pad 3: /C3 -> /D1
- U10 pad 4: /C4 -> /D2
- U10 pad 5: /C5 -> /D3
- U10 pad 6: (no net) -> /D4
- U10 pad 7: /R0 -> /D5
- U10 pad 8: GND -> /D6
- U10 pad 9: Net-(U10-Pad9) -> /D7
- U11 pad 1: /R2 -> GND
- U11 pad 10: /~RSTCOUNT -> /V3
- U11 pad 11: Net-(U10-Pad9) -> /V2
- U11 pad 12: GND -> /V1
- U11 pad 13: /DOTCLK -> Net-(R2-Pad2)
- U11 pad 14: /EXTEN -> /V0
- U11 pad 15: /R1 -> /~CSTART
- U11 pad 2: /R3 -> /V7
- U11 pad 3: /R4 -> /V6
- U11 pad 4: /R5 -> /V5
- U11 pad 5: /R6 -> /V4
- U11 pad 6: /R7 -> GND
- U11 pad 7: /R8 -> /DOTCLK
- U11 pad 9: (no net) -> +5V
- U3 pad 1: (no net) -> /VRAMWREN
- U3 pad 2: (no net) -> /EXTEN
- U3 pad 3: (no net) -> /VRAMOE
- U3 pad 4: (no net) -> /VRAMWREN
- U3 pad 5: (no net) -> /EXTWREN
- U3 pad 6: (no net) -> /~VRAMWE
- U4 pad 2: (no net) -> /HSYNC
- U4 pad 4: (no net) -> /VSYNC
- U4 pad 8: (no net) -> /~VRAMOE
- U4 pad 9: (no net) -> /VRAMOE
- U5 pad 5: (no net) -> /~EXTEN
- U5 pad 9: (no net) -> /EXTWREN
- U6 pad 1: /C5 -> +5V
- U6 pad 10: /R8 -> +5V
- U6 pad 11: /VD0 -> /~WRDATA
- U6 pad 12: /VD1 -> +5V
- U6 pad 13: /VS2 -> /~VRAMWREN
- U6 pad 14: GND -> +5V
- U6 pad 2: /R0 -> /WRPENDING
- U6 pad 3: /R1 -> /EXTEN
- U6 pad 4: /R2 -> +5V
- U6 pad 5: /R3 -> /VRAMWREN
- U6 pad 6: /R4 -> /~VRAMWREN
- U6 pad 7: /R5 -> GND
- U6 pad 8: /R6 -> (no net)
- U6 pad 9: /R7 -> /WRPENDING
- U7 pad 1: GND -> /C5
- U7 pad 10: GND -> /R8
- U7 pad 11: /VD7 -> /VD0
- U7 pad 12: /VD6 -> /VD1
- U7 pad 13: /VD5 -> /VD2
- U7 pad 14: /VD4 -> GND
- U7 pad 15: /VS3 -> /VD3
- U7 pad 16: /VS2 -> /VD4
- U7 pad 17: /VD1 -> /VD5
- U7 pad 18: /VD0 -> /VD6
- U7 pad 19: /~VIS -> /VD7
- U7 pad 2: /V0 -> /R0
- U7 pad 20: +5V -> GND
- U7 pad 3: /V1 -> /R1
- U7 pad 4: /V2 -> /R2
- U7 pad 5: /V3 -> /R3
- U7 pad 6: /V4 -> /R4
- U7 pad 7: /V5 -> /R5
- U7 pad 8: /V6 -> /R6
- U7 pad 9: /V7 -> /R7
- U8 pad 1: /~RSTCOUNT -> GND
- U8 pad 10: +5V -> GND
- U8 pad 11: /~CSTART -> /VD7
- U8 pad 12: /CDOT2 -> /VD6
- U8 pad 13: /CDOT1 -> /VD5
- U8 pad 14: /CDOT0 -> /VD4
- U8 pad 15: (no net) -> /VD3
- U8 pad 16: +5V -> /VD2
- U8 pad 2: /DOTCLK -> /V0
- U8 pad 3: +5V -> /V1
- U8 pad 4: GND -> /V2
- U8 pad 5: GND -> /V3
- U8 pad 6: +5V -> /V4
- U8 pad 7: +5V -> /V5
- U8 pad 8: GND -> /V6
- U8 pad 9: /~CSTART -> /V7
- U9 pad 1: GND -> /~RSTCOUNT
- U9 pad 10: /V3 -> +5V
- U9 pad 11: /V2 -> /~CSTART
- U9 pad 12: /V1 -> /CDOT2
- U9 pad 13: Net-(R2-Pad2) -> /CDOT1
- U9 pad 14: /V0 -> /CDOT0
- U9 pad 15: /~CSTART -> (no net)
- U9 pad 2: /V7 -> /DOTCLK
- U9 pad 3: /V6 -> +5V
- U9 pad 4: /V5 -> GND
- U9 pad 5: /V4 -> GND
- U9 pad 6: GND -> +5V
- U9 pad 7: /DOTCLK -> +5V
- U9 pad 9: +5V -> /~CSTART
Other:
- outline, holes or cut-outs redrawn
